File: DS2000.kicad_sch (KiCad schematic)
At the start: 36 parts, among them J1 USB_C_Receptacle_USB2.0_16P, SW1 SW_DPST_x2, SW2 SW_DPST_x2, SW3 SW_DPST_x2, U1 RP2040, U2 NCP1117-3.3_SOT223, U3 TPD2EUSB30, U4 W25Q128JVS, Y1 Crystal_GND2

Commit message: feat: redraw the schematic around the RP2350A
Rev A starts from a clean KiCad 10 project instead of patching the 2025 RP2040 draft, which is
kept in history at 7db9552.

- RP2350A with the on-chip switching regulator, decoupling, crystal, flash, BOOTSEL and RUN taken
  from Raspberry Pi's "Hardware design with RP2350" minimal design
- USB-C with CC resistors, a series PTC and USBLC6 ESD, AP2112K 3.3 V LDO
- Keys on GP0-GP2 to match the firmware's pins.h
- SK6812MINI-E under each key, fed from GP5 through a 74AHCT1G125 level shifter
- SWD on a Debug Probe JST-SH connector, four M2 mounting holes to GND

ERC reports no violations. The previous draft's defects (DVDD on 3.3 V, D+ on a SPICE ground,
bypassed fuse, wrong button GPIOs, missing BOOTSEL/SWD, sparse decoupling, oscillator footprint
on a crystal, LED currents) do not carry over.

Also drops the committed backups, fp-info-cache and .kicad_prl, and adds a .gitignore, README and
design notes. The layout starts once the board outline is agreed with the enclosure.
Parts:
- removed C1, C2: 10u, Capacitor_SMD:C_0402_1005Metric, symbol Device:C
- removed D1, D2: LED_KRGB, LED_SMD:LED_Avago_PLCC4_3.2x2.8mm_CW, symbol Device:LED_KRGB
- removed R1, R2: 27, Resistor_SMD:R_0402_1005Metric, symbol Device:R
- removed R11, R14: 82, Resistor_SMD:R_0402_1005Metric, symbol Device:R_Small
- removed R12, R13, R15, R16: 10, Resistor_SMD:R_0402_1005Metric, symbol Device:R_Small
- removed R5: 1k, Resistor_SMD:R_0402_1005Metric, symbol Device:R
- removed SW1, SW2, SW3: SW_DPST_x2, Button_Switch_Keyboard:SW_Cherry_MX_1.25u_Plate, symbol Switch:SW_DPST_x2
- removed U1: RP2040, Package_DFN_QFN:QFN-56-1EP_7x7mm_P0.4mm_EP3.2x3.2mm, symbol MCU_RaspberryPi:RP2040
- removed U2: NCP1117-3.3_SOT223, Package_TO_SOT_SMD:SOT-223-3_TabPin2, symbol Regulator_Linear:NCP1117-3.3_SOT223
- removed U3: TPD2EUSB30, Package_TO_SOT_SMD:Texas_DRT-3, symbol Power_Protection:TPD2EUSB30
- removed U4: W25Q128JVS, Package_SO:SOIC-8_5.3x5.3mm_P1.27mm, symbol Memory_Flash:W25Q128JVS
- removed Y1: Crystal_GND2, Oscillator:Oscillator_SMD_EuroQuartz_XO32-4Pin_3.2x2.5mm_RotB, symbol Device:Crystal_GND2
- added C1, C2: 10u, Capacitor_SMD:C_0805_2012Metric, symbol Device:C_Small
- added C10, C11, C12, C13, C14, C15, C16, C19, C20, C21, C22, C23, C9: 100n, Capacitor_SMD:C_0402_1005Metric, symbol Device:C_Small
- added C17, C18: 15p, Capacitor_SMD:C_0402_1005Metric, symbol Device:C_Small
- added D1, D2, D3: SK6812MINI-E, LED_SMD:LED_SK6812MINI-E_3.2x2.8mm_P1.5mm_ReverseMount, symbol LED:SK6812MINI-E
- added H1, H2, H3, H4: M2, MountingHole:MountingHole_2.2mm_M2_Pad_Via, symbol Mechanical:MountingHole_Pad
- added J2: SWD, Connector_JST:JST_SH_SM03B-SRSS-TB_1x03-1MP_P1.00mm_Horizontal, symbol Connector_Generic:Conn_01x03
- added L1: 3.3u, Inductor_SMD:L_Murata_DFE201610P, symbol Device:L_Small
- added R1, R2: 5.1k, Resistor_SMD:R_0402_1005Metric, symbol Device:R_Small
- added R5: 33, Resistor_SMD:R_0402_1005Metric, symbol Device:R_Small
- added SW1: MUTE, Button_Switch_Keyboard:SW_Cherry_MX_1.00u_PCB, symbol Switch:SW_Push
- added SW2: DEAFEN, Button_Switch_Keyboard:SW_Cherry_MX_1.00u_PCB, symbol Switch:SW_Push
- added SW3: DISCONNECT, Button_Switch_Keyboard:SW_Cherry_MX_1.00u_PCB, symbol Switch:SW_Push
- added SW4: BOOTSEL, Button_Switch_SMD:SW_Push_1P1T_XKB_TS-1187A, symbol Switch:SW_Push
- added SW5: RESET, Button_Switch_SMD:SW_Push_1P1T_XKB_TS-1187A, symbol Switch:SW_Push
- added U1: USBLC6-2SC6, Package_TO_SOT_SMD:SOT-23-6, symbol Power_Protection:USBLC6-2SC6
- added U2: AP2112K-3.3, Package_TO_SOT_SMD:SOT-23-5, symbol Regulator_Linear:AP2112K-3.3
- added U3: RP2350A, Package_DFN_QFN:QFN-60-1EP_7x7mm_P0.4mm_EP3.4x3.4mm_ThermalVias, symbol MCU_RaspberryPi:RP2350A
- added U4: W25Q32JVSS, Package_SO:SOIC-8_5.3x5.3mm_P1.27mm, symbol Memory_Flash:W25Q32JVSS
- added U5: 74AHCT1G125, Package_TO_SOT_SMD:SOT-353_SC-70-5, symbol 74xGxx:74AHCT1G125
- added Y1: 12MHz, Crystal:Crystal_SMD_3225-4Pin_3.2x2.5mm, symbol Device:Crystal_GND24_Small
- C3: value 100n -> 4.7u; Note (none) -> VREG output cap, layout per RP2350 guide
- C4: value 1u -> 4.7u; Note (none) -> VREG_VIN
- C5: value 1u -> 4.7u; Note (none) -> VREG_AVDD RC filter
- C6, C7: value 15p -> 100n
- F1: value Polyfuse_Small -> 500mA hold; footprint Diode_SMD:Littelfuse_PolyZen-LS -> Fuse:Fuse_1206_3216Metric; MPN (none) -> 1206L050YR; Manufacturer (none) -> Littelfuse
- J1: value USB_C_Receptacle_USB2.0_16P -> USB-C; footprint Connector_USB:USB_C_Receptacle_Palconn_UTC16-G -> Connector_USB:USB_C_Receptacle_HRO_TYPE-C-31-M-12; MPN (none) -> TYPE-C-31-M-12; Manufacturer (none) -> Korean Hroparts Elec
- R10: value 10k -> 100; Note (none) -> Damping, place near D1
- R3, R4: value 5.1k -> 27; Note (none) -> Place close to U3
- R6, R8: value 10k -> 1k
- R7: Note (none) -> DNF: only needed with other flash parts; now not fitted
Connections:
- net GND: now also C4.2, C5.2, C6.2, J1.SH (SHIELD), C1.2, C10.2, C11.2, C12.2, C13.2, C14.2, C15.2, C16.2, C17.2, C18.2, C19.2, C2.2, C20.2, C21.2, C22.2, C23.2, C9.2, D1.1 (VSS), D2.1 (VSS), D3.1 (VSS), H1.1, H2.1, H3.1, H4.1, J2.2 (Pin_2), R1.2, R2.2, SW1.2, SW2.2, SW3.2, SW4.2, SW5.2, U1.2 (GND), U2.2 (GND), U3.47 (VREG_PGND), U3.61 (GND), U4.4 (GND), U5.1, U5.3 (GND), Y1.2 (G), Y1.4 (G); no longer C4.1, C5.1, C6.1, J1.S1 (SHIELD), R3.2
- net +3V3: now reaches C7.1
- net +3V3: now also C4.1, C6.1, C8.1, R7.1, R9.1, C10.1, C11.1, C15.1, C16.1, C19.1, C2.1, C9.1, R5.1, U2.5 (VOUT), U3.1 (IOVDD), U3.11 (IOVDD), U3.20 (IOVDD), U3.30 (IOVDD), U3.38 (IOVDD), U3.44 (ADC_AVDD), U3.45 (IOVDD), U3.49 (VREG_VIN), U3.53 (USB_OTP_VDD), U3.54 (QSPI_IOVDD), U4.8 (VCC)
- net BOOTSEL: now reaches R8.2
- net BOOTSEL: now also SW4.1
- net RUN: now reaches R9.2
- net RUN: now also SW5.1, U3.26 (RUN)
- net XTAL_OUT: now reaches R6.2
- net XTAL_OUT: now also C18.1, Y1.3
- net LED_DIN: now reaches R10.2
- net LED_DIN: now also D1.2 (DIN)
- net CC1: now reaches J1.A5 (CC1)
- net CC1: now also R1.1; no longer R3.1
- net USB_CONN_DM: now reaches J1.A7 (D-), J1.B7 (D-)
- net USB_CONN_DM: now also R4.1, U1.3 (I/O2), U1.4 (I/O2)
- net VBUS: now reaches F1.1, J1.A4 (VBUS), J1.A9 (VBUS), J1.B4 (VBUS), J1.B9 (VBUS)
- net VBUS: no longer F1.2
- net CC2: now reaches J1.B5 (CC2)
- net CC2: now also R2.1; no longer R4.1
- net USB_DM: now reaches R4.2
- net USB_DM: now also U3.51 (USB_DM)
- net 0 renamed USB_CONN_DP
- net USB_CONN_DP: now also R3.1, U1.1 (I/O1), U1.6 (I/O1)
- removed net 3.3V: C3.1, C4.2, C8.1, R10.1, R6.1, R7.2, R8.1, R9.1
- new net +1V1: C12.1, C13.1, C14.1, C3.1, L1.2, U3.23 (DVDD), U3.39 (DVDD), U3.50 (VREG_FB), U3.6 (DVDD)
- new net +5V: C1.1, C20.1, C21.1, C22.1, C23.1, D1.3 (VDD), D2.3 (VDD), D3.3 (VDD), F1.2, U1.5 (VBUS), U2.1 (VIN), U2.3 (EN), U5.5 (VCC)
- new net KEY_DEAFEN: SW2.1, U3.3 (GPIO1)
- new net KEY_DISCONNECT: SW3.1, U3.4 (GPIO2)
- new net KEY_MUTE: SW1.1, U3.2 (GPIO0)
- new net LED_D1_D2: D1.4 (DOUT), D2.2 (DIN)
- new net LED_D2_D3: D2.4 (DOUT), D3.2 (DIN)
- new net LED_DIN_3V3: U3.8 (GPIO5), U5.2
- new net LED_DIN_5V: R10.1, U5.4
- new net QSPI_SCLK: U3.56 (QSPI_SCLK), U4.6 (CLK)
- new net QSPI_SD0: U3.57 (QSPI_SD0), U4.5 (DI/IO_{0})
- new net QSPI_SD1: U3.59 (QSPI_SD1), U4.2 (DO/IO_{1})
- new net QSPI_SD2: U3.58 (QSPI_SD2), U4.3 (~{WP}/IO_{2})
- new net QSPI_SD3: U3.55 (QSPI_SD3), U4.7 (~{HOLD}/~{RESET}/IO_{3})
- new net QSPI_SS: R7.2, R8.1, U3.60 (~{QSPI_SS}), U4.1 (~{CS})
- new net SWCLK: J2.1 (Pin_1), U3.24 (SWCLK)
- new net SWDIO: J2.3 (Pin_3), U3.25 (SWDIO)
- new net USB_DP: R3.2, U3.52 (USB_DP)
- new net VREG_AVDD: C5.1, R5.2, U3.46 (VREG_AVDD)
- new net VREG_LX: L1.1, U3.48 (VREG_LX)
- new net XIN: C17.1, U3.21 (XIN), Y1.1
- new net XOUT: R6.1, U3.22 (XOUT)
- no-connect marks 0 -> 30
Other:
- note added: "Decoupling at the pins: C6-C11 IOVDD, C12-C14 DVDD, C15 ADC_AVDD, C16 USB_OTP_VDD+QSPI_IOVDD"
- note added: "Keys (GP0-GP2, internal pull-ups) and per-key SK6812MINI-E"
- note added: "RP2350A, core regulator, crystal, flash"
- note added: "Reset, SWD, mounting"
- note added: "USB-C input, protection, 3.3 V LDO"
- company: (none) -> Mechardo Labs
- title: (none) -> DS-2000

Commit message: feat: draw each stage in its own wired block and add USB wire pads
The schematic is now laid out by stage (USB input, 3.3 V regulator, reset, mounting holes, RP2350A
supplies, RP2350A, flash and BOOTSEL, crystal and SWD, keys, key LEDs, decoupling), each in a
titled box and wired internally. Net labels remain only where a signal leaves its stage. The flash
is mirrored so the six QSPI lines run straight into the RP2350A, and the core regulator is wired
directly onto the MCU's supply pins.

J3 adds four bare 2.54 mm holes (VBUS, D-, D+, GND) for soldering a USB cable instead of fitting
the receptacle. They sit upstream of the fuse and the ESD, so a hard-wired cable is protected the
same way.

The generator now declares every part's connectivity and check_netlist.py compares it with
KiCad's netlist export; both that and ERC pass. Design notes record the RP2350A on show on the top
side, the 5-pin switch footprint and the firmware work in DS-2000-Firmware#13.
Parts:
- added J3: USB wire, Connector_PinHeader_2.54mm:PinHeader_1x04_P2.54mm_Vertical, symbol Connector_Generic:Conn_01x04
- C10, C11, C6, C7, C8, C9: Note (none) -> IOVDD
- C12, C13, C14: Note (none) -> DVDD
- C15: Note (none) -> ADC_AVDD
- C16: Note (none) -> USB_OTP+QSPI_IOVDD
- C3: Note VREG output cap, layout per RP2350 guide -> VREG output cap
- C5, R5: Note VREG_AVDD RC filter -> (none)
- L1: Note Polarity-marked inductor; orientation matters. Verify pads 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 -> Polarity-marked; orientation and layout per RP2350 guide. V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
- R10: Note Damping, place near D1 -> Damping, near D1
- R7: Note DNF: only needed with other flash parts -> DNF, only for other flash parts
- U5: Note 3.3 V -> 5 V level shift for the LED data line -> (none)
Connections:
- net GND: now also R1.1, R2.1, SW4.1, J3.4 (Pin_4); no longer R1.2, R2.2, SW4.2
- net USB_CONN_DM: now also U1.1 (I/O1), U1.6 (I/O1), J3.2 (Pin_2); no longer U1.3 (I/O2), U1.4 (I/O2)
- net USB_CONN_DP: now also U1.3 (I/O2), U1.4 (I/O2), J3.3 (Pin_3); no longer U1.1 (I/O1), U1.6 (I/O1)
- net VBUS: now also J3.1 (Pin_1)
- net BOOTSEL: no longer names the net of R8.2
- net BOOTSEL: now also R7.2, U3.60 (~{QSPI_SS}), U4.1 (~{CS}); no longer SW4.1
- net CC1: no longer names the net of J1.A5 (CC1)
- net CC1: now also R1.2; no longer R1.1
- net CC2: no longer names the net of J1.B5 (CC2)
- net CC2: now also R2.2; no longer R2.1
- net KEY_DEAFEN: no longer names the net of SW2.1, U3.3 (GPIO1)
- net KEY_DISCONNECT: no longer names the net of SW3.1, U3.4 (GPIO2)
- net KEY_MUTE: no longer names the net of SW1.1, U3.2 (GPIO0)
- net LED_D1_D2: no longer names the net of D1.4 (DOUT), D2.2 (DIN)
- net LED_D2_D3: no longer names the net of D2.4 (DOUT), D3.2 (DIN)
- net LED_DIN: no longer names the net of D1.2 (DIN), R10.2
- net LED_DIN_3V3: no longer names the net of U3.8 (GPIO5), U5.2
- net LED_DIN_5V: no longer names the net of R10.1, U5.4
- net QSPI_SCLK: no longer names the net of U3.56 (QSPI_SCLK), U4.6 (CLK)
- net QSPI_SD0: no longer names the net of U3.57 (QSPI_SD0), U4.5 (DI/IO_{0})
- net QSPI_SD1: no longer names the net of U3.59 (QSPI_SD1), U4.2 (DO/IO_{1})
- net QSPI_SD2: no longer names the net of U3.58 (QSPI_SD2), U4.3 (~{WP}/IO_{2})
- net QSPI_SD3: no longer names the net of U3.55 (QSPI_SD3), U4.7 (~{HOLD}/~{RESET}/IO_{3})
- removed net QSPI_SS: R7.2, R8.1, U3.60 (~{QSPI_SS}), U4.1 (~{CS})
- net SWCLK: no longer names the net of J2.1 (Pin_1), U3.24 (SWCLK)
- net SWDIO: no longer names the net of J2.3 (Pin_3), U3.25 (SWDIO)
- net VREG_AVDD: no longer names the net of C5.1, R5.2, U3.46 (VREG_AVDD)
- net VREG_LX: no longer names the net of L1.1, U3.48 (VREG_LX)
- net XIN: no longer names the net of C17.1, U3.21 (XIN), Y1.1
- net XOUT: no longer names the net of R6.1
- net XOUT: now also C18.1, Y1.3; no longer U3.22 (XOUT)
- removed net XTAL_OUT: C18.1, R6.2, Y1.3
- new net: R8.1, SW4.2
- new net: R6.2, U3.22 (XOUT)
Other:
- note added: "12 MHz crystal, SWD"
- note added: "3.3 V regulator"
- note added: "C4 VREG_VIN · C6-C11 IOVDD x6 · C12-C14 DVDD x3 · C15 ADC_AVDD · C16 USB_OTP_VDD + QSPI_IOVDD (shared, as in the reference)"
- note added: "CC 5.1k: USB device (UFP). U1 at the connector, R3/R4 next to the RP2350. J3: optional soldered cable."
- note added: "Core regulator: layout exactly as the RP2350 guide"
- note added: "D1 mute, D2 deafen, D3 disconnect (reverse-mounted under each key). One 100n per LED."
- note added: "Decoupling, placed at the pins"
- note added: "EN tied to VIN: always on. 250 mV dropout."
- note added: "GP0-GP2, internal pull-ups"
- note added: "Hold BOOTSEL while resetting to enter USB boot."
- note added: "Key LEDs: 3.3 V -> 5 V level shift, SK6812MINI-E chain"
- note added: "Keys"
- note added: "Mounting holes (PCB corners, to GND)"
- note added: "QSPI flash and BOOTSEL"
- note added: "RP2350A"
- note added: "RP2350A supplies"
- note added: "Reset"
- note added: "USB-C input, fuse, ESD and wire pads"
- note removed: "Decoupling at the pins: C6-C11 IOVDD, C12-C14 DVDD, C15 ADC_AVDD, C16 USB_OTP_VDD+QSPI_IOVDD"
- note removed: "Keys (GP0-GP2, internal pull-ups) and per-key SK6812MINI-E"
- note removed: "RP2350A, core regulator, crystal, flash"
- note removed: "Reset, SWD, mounting"
- note removed: "USB-C input, protection, 3.3 V LDO"
