File: DS2000.kicad_pcb (KiCad board)
At the start: 4 copper layers, 72 x 46 mm, 58 parts, among them J1 USB-C, J3 USB wire, SW1 MUTE, SW2 DEAFEN, SW3 DISCONNECT, U1 USBLC6-2SC6, U2 AP2112K-3.3, U3 RP2350A, U4 W25Q32JVSS, U5 74AHCT1G125, Y1 12MHz

Commit message: feat: keep autorouted tracks off the visible top face
The board is the product's top face, but Freerouting used F.Cu freely: +5V to the LEDs, the debug
lines, RUN and the key lines ran across the key area and beside the logos. top_keepout.py now puts a
track keepout on F.Cu over everything but the component strip around the RP2350A while the
autorouter runs, and takes it out afterwards, so every longer run goes on B.Cu.

F.Cu tracks: 399 -> 344 mm, all inside the strip; the key area and the sides carry none. XIN, QSPI
SCLK, VREG_LX and USB D+/D- between U3 and R3/R4 are unchanged.
Routing:
- net Net-(JP1-B): track 40.3 -> 101.2 mm, vias 1 -> 3
- net VBUS: track 34.4 -> 83.9 mm, vias 1 -> 6
- net Net-(U3-SWCLK): track 22.6 -> 41.6 mm
- net +5V: track 115.1 -> 96.9 mm, vias 5 -> 4
- net /USB_CONN_DM: track 38.5 -> 51.7 mm, vias 1 -> 2
- net Net-(U3-GPIO1): track 22.6 -> 17.5 mm, vias 2 -> 1
- net Net-(U3-SWDIO): track 29.9 -> 34.5 mm
- net Net-(U3-~{QSPI_SS}): track 20.5 -> 24.5 mm, vias 2 -> 0
- net /USB_CONN_DP: track 30.9 -> 34.0 mm, vias 1 -> 2
- net Net-(U3-GPIO0): track 20.1 -> 23.1 mm
- net Net-(U3-GPIO2): track 31.1 -> 28.4 mm, vias 2 -> 1
- net /RUN: track 33.4 -> 31.4 mm
- net +1V1: track 37.6 -> 35.7 mm
- net Net-(J1-CC2): track 9.32 -> 7.35 mm
- net Net-(J1-CC1): track 9.60 -> 8.21 mm
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